Commit message: add lidar to macnav_description

File: ws/src/macnav_description/urdf/common_properties.xacro (robot description, xacro)
@@ -1,4 +1,9 @@
 <?xml version="1.0"?>
 <robot xmlns:xacro="http://www.ros.org/wiki/xacro">
+    <xacro:property name="chassis_length" value="0.370" />
+    <xacro:property name="chassis_width" value="0.250" />
+    <xacro:property name="chassis_height" value="0.160" />
+    <xacro:property name="wheel_radius" value="0.041" />
+    <xacro:property name="wheel_length" value="0.032" />
     <material name="red">
         <color rgba="0.5 0 0 1"/>

File: ws/src/macnav_description/urdf/macnav.urdf.xacro (robot description, xacro)
@@ -2,4 +2,5 @@
 <robot name="macnav" xmlns:xacro="http://www.ros.org/wiki/xacro">
     <xacro:include filename="common_properties.xacro" />
-    <xacro:include filename="macnav.xacro" />
+    <xacro:include filename="macnav_base.xacro" />
+    <xacro:include filename="macnav_lidar.xacro"/>
 </robot>

File: ws/src/macnav_description/urdf/macnav_base.xacro (robot description, xacro)
@@ -1,9 +1,4 @@
 <?xml version="1.0" ?>
 <robot xmlns:xacro="http://www.ros.org/wiki/xacro">
-    <xacro:property name="chassis_length" value="0.370" />
-    <xacro:property name="chassis_width" value="0.250" />
-    <xacro:property name="chassis_height" value="0.160" />
-    <xacro:property name="wheel_radius" value="0.041" />
-    <xacro:property name="wheel_length" value="0.032" />
     <link name="base_link"/>
     <link name="chassis">

Commit message: add axle and universal steer joints to urdf

File: ws/src/macnav_description/urdf/common_properties.xacro (robot description, xacro)
@@ -1,5 +1,4 @@
 <?xml version="1.0"?>
 <robot xmlns:xacro="http://www.ros.org/wiki/xacro">
-<<<<<<< HEAD
     <xacro:property name="chassis_length" value="0.370" />
     <xacro:property name="chassis_width" value="0.250" />
@@ -7,6 +6,4 @@
     <xacro:property name="wheel_radius" value="0.041" />
     <xacro:property name="wheel_length" value="0.032" />
-=======
->>>>>>> 12dae00a0c536b2e3cf805fae25f64fdce2a2b12
     <material name="red">
         <color rgba="0.5 0 0 1"/>

File: ws/src/macnav_description/urdf/macnav.urdf.xacro (robot description, xacro)
@@ -2,9 +2,5 @@
 <robot name="macnav" xmlns:xacro="http://www.ros.org/wiki/xacro">
     <xacro:include filename="common_properties.xacro" />
-<<<<<<< HEAD
     <xacro:include filename="macnav_base.xacro" />
     <xacro:include filename="macnav_lidar.xacro"/>
-=======
-    <xacro:include filename="macnav.xacro" />
->>>>>>> 12dae00a0c536b2e3cf805fae25f64fdce2a2b12
 </robot>

File: ws/src/macnav_description/urdf/macnav_base.xacro (robot description, xacro)
@@ -36,4 +36,13 @@
     <xacro:wheel_link prefix="rear_left"/>
     <xacro:wheel_link prefix="rear_right"/>
+    <link name="steer_link">
+        <visual>
+            <origin xyz="0 0 0" rpy="0 0 0"/>
+            <geometry>
+                <box size="${chassis_height/10} ${chassis_height/10} ${chassis_height/10}"/>
+            </geometry>
+        </visual>
+        <xacro:box_inertia m="0.01" l="${chassis_height/10}" w="${chassis_height/10}" h="${chassis_height/10}" xyz="0 0 0" rpy="0 0 0"/>
+    </link>
     <link name="front_left_steer_link">
         <visual>
@@ -54,4 +63,15 @@
         <xacro:box_inertia m="0.01" l="${chassis_height/10}" w="${chassis_height/10}" h="${chassis_height/10}" xyz="0 0 0" rpy="0 0 0"/>
     </link>
+    <link name="rear_axle_link">
+        <visual>
+            <geometry>
+                <cylinder radius="${wheel_radius/2}" length="${chassis_width}" />
+            </geometry>
+            <origin xyz="0 0 0" rpy="${pi / 2.0} 0 0" />
+               <material name="blue" />
+        </visual>
+        <xacro:cylinder_inertia m="1.0" r="${wheel_radius/2}" h="${chassis_width}"
+                            xyz="0 0 0" rpy="${pi / 2.0} 0 0" />
+    </link>
     <joint name="base_joint" type="fixed">
         <parent link="base_link"/>
@@ -59,5 +79,13 @@
         <origin xyz="0 0 ${wheel_radius/2}" rpy="0 0 0"/>
     </joint>
+    <joint name="steer_joint" type="revolute">
+        <parent link="chassis"/>
+        <child link="steer_link"/>
+        <origin xyz="${chassis_length - (3*chassis_length/5)} 0 0" rpy="0 0 0"/>
+        <axis xyz="0 0 1"/>
+        <limit effort="100" lower="-0.5" upper="0.5" velocity="10"/>
+    </joint>
     <joint name="front_left_steer_chassis_joint" type="revolute">
+        <mimic joint="steer_joint"/>
         <parent link="chassis"/>
         <child link="front_left_steer_link"/>
@@ -73,4 +101,5 @@
     </joint>
     <joint name="front_right_steer_chassis_joint" type="revolute">
+        <mimic joint="steer_joint"/>
         <parent link="chassis"/>
         <child link="front_right_steer_link"/>
@@ -85,15 +114,19 @@
         <axis xyz="0 1 0"/>
     </joint>
-    <joint name="rear_left_wheel_chassis_joint" type="continuous">
+    <joint name="rear_axle_joint" type="continuous">
         <parent link="chassis"/>
-        <child link="rear_left_wheel_link"/>
-        <origin xyz="${-chassis_length + (3*chassis_length/5)} ${(chassis_width + wheel_length) / 2} 0" rpy="0 0 0"/>
+        <child link="rear_axle_link"/>
+        <origin xyz="${-chassis_length + (3*chassis_length/5)} 0 0" rpy="0 0 0"/>
         <axis xyz="0 1 0"/>
     </joint>
-    <joint name="rear_right_wheel_chassis_joint" type="continuous">
-        <parent link="chassis"/>
+    <joint name="rear_left_wheel_chassis_joint" type="fixed">
+        <parent link="rear_axle_link"/>
+        <child link="rear_left_wheel_link"/>
+        <origin xyz="0 ${(chassis_width + wheel_length) / 2} 0" rpy="0 0 0"/>
+    </joint>
+    <joint name="rear_right_wheel_chassis_joint" type="fixed">
+        <parent link="rear_axle_link"/>
         <child link="rear_right_wheel_link"/>
-        <origin xyz="${-chassis_length + (3*chassis_length/5)} ${-(chassis_width + wheel_length) / 2} 0" rpy="0 0 0"/>
-        <axis xyz="0 1 0"/>
+        <origin xyz="0 ${-(chassis_width + wheel_length) / 2} 0" rpy="0 0 0"/>
     </joint>
 </robot>
