Commit message: initial dev of odom publishing

File: remote_setup/ws/src/macnav_description/urdf/common_properties.xacro (robot description, xacro)
@@ -4,5 +4,5 @@
     <xacro:property name="chassis_width" value="0.250" />
     <xacro:property name="chassis_height" value="0.160" />
-    <xacro:property name="wheel_radius" value="0.041" />
+    <xacro:property name="wheel_radius" value="0.042525" />
     <xacro:property name="wheel_length" value="0.032" />
     <material name="red">
