Commit message: SLAM MAPS WORKING

File: remote_setup/ws/src/macnav_description/urdf/macnav_base.xacro (robot description, xacro)
@@ -2,4 +2,5 @@
 <robot xmlns:xacro="http://www.ros.org/wiki/xacro">
     <link name="base_link"/>
+    <link name="base_footprint"/>
     <link name="chassis">
         <visual>
@@ -74,4 +75,9 @@
                             xyz="0 0 0" rpy="${pi / 2.0} 0 0" />
     </link>
+    <joint name="base_footprint_joint" type="fixed">
+        <parent link="base_link"/>
+        <child link="base_footprint"/>
+        <origin xyz="0 0 0" rpy="0 0 0"/>
+    </joint>
     <joint name="base_joint" type="fixed">
         <parent link="base_link"/>
