Commit message: finish odom tf

File: remote_setup/ws/install/macnav_description/share/macnav_description/urdf/common_properties.xacro (robot description, xacro)
@@ -1,47 +1 @@
-<?xml version="1.0"?>
-<robot xmlns:xacro="http://www.ros.org/wiki/xacro">
-    <xacro:property name="chassis_length" value="0.370" />
-    <xacro:property name="chassis_width" value="0.250" />
-    <xacro:property name="chassis_height" value="0.160" />
-    <xacro:property name="wheel_radius" value="0.042525" />
-    <xacro:property name="wheel_length" value="0.032" />
-    <material name="red">
-        <color rgba="0.5 0 0 1"/>
-    </material>
-    <material name="green">
-        <color rgba="0 0.5 0 1"/>
-    </material>
-    <material name="blue">
-        <color rgba="0 0 0.5 1"/>
-    </material>
-    <material name="grey">
-        <color rgba="0.5 0.5 0.5 1" />
-    </material>
-    <xacro:macro name="box_inertia" params="m l w h xyz rpy">
-        <inertial>
-            <origin xyz="${xyz}" rpy="${rpy}" />
-            <mass value="${m}" />
-            <inertia ixx="${(m/12) * (h*h + l*l)}" ixy="0" ixz="0"
-                     iyy="${(m/12) * (w*w + l*l)}" iyz="0"
-                     izz="${(m/12) * (w*w + h*h)}" />
-        </inertial>
-    </xacro:macro>
-    <xacro:macro name="cylinder_inertia" params="m r h xyz rpy">
-        <inertial>
-            <origin xyz="${xyz}" rpy="${rpy}" />
-            <mass value="${m}" />
-            <inertia ixx="${(m/12) * (3*r*r + h*h)}" ixy="0" ixz="0"
-                     iyy="${(m/12) * (3*r*r + h*h)}" iyz="0"
-                     izz="${(m/2) * (r*r)}" />
-        </inertial>
-    </xacro:macro>
-    <xacro:macro name="sphere_inertia" params="m r xyz rpy">
-        <inertial>
-            <origin xyz="${xyz}" rpy="${rpy}" />
-            <mass value="${m}" />
-            <inertia ixx="${(2/5) * m * r * r}" ixy="0" ixz="0"
-                     iyy="${(2/5) * m * r * r}" iyz="0"
-                     izz="${(2/5) * m * r * r}" />
-        </inertial>
-    </xacro:macro>
-</robot>
+/mac_remote/ws/src/macnav_description/urdf/common_properties.xacro

File: remote_setup/ws/install/macnav_description/share/macnav_description/urdf/macnav.urdf.xacro (robot description, xacro)
@@ -1,6 +1 @@
-<?xml version="1.0"?>
-<robot name="macnav" xmlns:xacro="http://www.ros.org/wiki/xacro">
-    <xacro:include filename="common_properties.xacro" />
-    <xacro:include filename="macnav_base.xacro" />
-    <xacro:include filename="macnav_lidar.xacro"/>
-</robot>
+/mac_remote/ws/src/macnav_description/urdf/macnav.urdf.xacro

File: remote_setup/ws/install/macnav_description/share/macnav_description/urdf/macnav_base.xacro (robot description, xacro)
@@ -1,132 +1 @@
-<?xml version="1.0" ?>
-<robot xmlns:xacro="http://www.ros.org/wiki/xacro">
-    <link name="base_link"/>
-    <link name="chassis">
-        <visual>
-            <geometry>
-                <box size="${chassis_length} ${chassis_width} ${chassis_height}" />
-            </geometry>
-            <origin xyz="0 0 ${chassis_height / 2.0}" rpy="0 0 0" />
-            <material name="red"/>
-        </visual>
-        <collision>
-            <origin xyz="0 0 0" rpy="0 0 0"/>
-            <geometry>
-                <box size="${chassis_length} ${chassis_width} ${chassis_height}" />
-            </geometry>
-        </collision>
-        <xacro:box_inertia m="5.0" l="${chassis_length}" w="${chassis_width}" h="${chassis_height}"
-                    xyz="0 0 ${chassis_height / 2.0}" rpy="0 0 0" />
-    </link>
-    <xacro:macro name="wheel_link" params="prefix">
-        <link name="${prefix}_wheel_link">
-            <visual>
-                <geometry>
-                    <cylinder radius="${wheel_radius}" length="${wheel_length}" />
-                </geometry>
-                <origin xyz="0 0 0" rpy="${pi / 2.0} 0 0" />
-                <material name="blue" />
-            </visual>
-            <xacro:cylinder_inertia m="1.0" r="${wheel_radius}" h="${wheel_length}"
-                                    xyz="0 0 0" rpy="${pi / 2.0} 0 0" />
-        </link>
-    </xacro:macro>
-    <xacro:wheel_link prefix="front_left"/>
-    <xacro:wheel_link prefix="front_right"/>
-    <xacro:wheel_link prefix="rear_left"/>
-    <xacro:wheel_link prefix="rear_right"/>
-    <link name="steer_link">
-        <visual>
-            <origin xyz="0 0 0" rpy="0 0 0"/>
-            <geometry>
-                <box size="${chassis_height/10} ${chassis_height/10} ${chassis_height/10}"/>
-            </geometry>
-        </visual>
-        <xacro:box_inertia m="0.01" l="${chassis_height/10}" w="${chassis_height/10}" h="${chassis_height/10}" xyz="0 0 0" rpy="0 0 0"/>
-    </link>
-    <link name="front_left_steer_link">
-        <visual>
-            <origin xyz="0 0 0" rpy="0 0 0"/>
-            <geometry>
-                <box size="${chassis_height/10} ${chassis_height/10} ${chassis_height/10}"/>
-            </geometry>
-        </visual>
-        <xacro:box_inertia m="0.01" l="${chassis_height/10}" w="${chassis_height/10}" h="${chassis_height/10}" xyz="0 0 0" rpy="0 0 0"/>
-    </link>
-    <link name="front_right_steer_link">
-        <visual>
-            <origin xyz="0 0 0" rpy="0 0 0"/>
-            <geometry>
-                <box size="${chassis_height/10} ${chassis_height/10} ${chassis_height/10}"/>
-            </geometry>
-        </visual>
-        <xacro:box_inertia m="0.01" l="${chassis_height/10}" w="${chassis_height/10}" h="${chassis_height/10}" xyz="0 0 0" rpy="0 0 0"/>
-    </link>
-    <link name="rear_axle_link">
-        <visual>
-            <geometry>
-                <cylinder radius="${wheel_radius/2}" length="${chassis_width}" />
-            </geometry>
-            <origin xyz="0 0 0" rpy="${pi / 2.0} 0 0" />
-               <material name="blue" />
-        </visual>
-        <xacro:cylinder_inertia m="1.0" r="${wheel_radius/2}" h="${chassis_width}"
-                            xyz="0 0 0" rpy="${pi / 2.0} 0 0" />
-    </link>
-    <joint name="base_joint" type="fixed">
-        <parent link="base_link"/>
-        <child link="chassis"/>
-        <origin xyz="0 0 ${wheel_radius/2}" rpy="0 0 0"/>
-    </joint>
-    <joint name="steer_joint" type="revolute">
-        <parent link="chassis"/>
-        <child link="steer_link"/>
-        <origin xyz="${chassis_length - (3*chassis_length/5)} 0 0" rpy="0 0 0"/>
-        <axis xyz="0 0 1"/>
-        <limit effort="100" lower="-0.5" upper="0.5" velocity="10"/>
-    </joint>
-    <joint name="front_left_steer_chassis_joint" type="revolute">
-        <mimic joint="steer_joint"/>
-        <parent link="chassis"/>
-        <child link="front_left_steer_link"/>
-        <origin xyz="${chassis_length - (3*chassis_length/5)} ${(chassis_width + wheel_length) / 2} 0" rpy="0 0 0"/>
-        <axis xyz="0 0 1"/>
-        <limit effort="100" lower="-0.5" upper="0.5" velocity="10"/>
-    </joint>
-    <joint name="front_left_wheel_steer_joint" type="continuous">
-        <parent link="front_left_steer_link"/>
-        <child link="front_left_wheel_link"/>
-        <origin xyz="0 0 0" rpy="0 0 0"/>
-        <axis xyz="0 1 0"/>
-    </joint>
-    <joint name="front_right_steer_chassis_joint" type="revolute">
-        <mimic joint="steer_joint"/>
-        <parent link="chassis"/>
-        <child link="front_right_steer_link"/>
-        <origin xyz="${chassis_length - (3*chassis_length/5)} ${-(chassis_width + wheel_length) / 2} 0" rpy="0 0 0"/>
-        <axis xyz="0 0 1"/>
-        <limit effort="100" lower="-0.5" upper="0.5" velocity="10"/>
-    </joint>
-    <joint name="front_right_wheel_steer_joint" type="continuous">
-        <parent link="front_right_steer_link"/>
-        <child link="front_right_wheel_link"/>
-        <origin xyz="0 0 0" rpy="0 0 0"/>
-        <axis xyz="0 1 0"/>
-    </joint>
-    <joint name="rear_axle_joint" type="continuous">
-        <parent link="chassis"/>
-        <child link="rear_axle_link"/>
-        <origin xyz="${-chassis_length + (3*chassis_length/5)} 0 0" rpy="0 0 0"/>
-        <axis xyz="0 1 0"/>
-    </joint>
-    <joint name="rear_left_wheel_chassis_joint" type="fixed">
-        <parent link="rear_axle_link"/>
-        <child link="rear_left_wheel_link"/>
-        <origin xyz="0 ${(chassis_width + wheel_length) / 2} 0" rpy="0 0 0"/>
-    </joint>
-    <joint name="rear_right_wheel_chassis_joint" type="fixed">
-        <parent link="rear_axle_link"/>
-        <child link="rear_right_wheel_link"/>
-        <origin xyz="0 ${-(chassis_width + wheel_length) / 2} 0" rpy="0 0 0"/>
-    </joint>
-</robot>
+/mac_remote/ws/src/macnav_description/urdf/macnav_base.xacro

File: remote_setup/ws/install/macnav_description/share/macnav_description/urdf/macnav_lidar.xacro (robot description, xacro)
@@ -1,23 +1 @@
-<?xml version="1.0"?>
-<robot xmlns:xacro="http://www.ros.org/wiki/xacro">
-    <joint name="laser_joint" type="fixed">
-        <parent link="chassis"/>
-        <child link="laser_frame"/>
-        <origin xyz="0 0 ${9 / 8 * chassis_height }" rpy="0 0 0"/>
-    </joint>
-    <link name="laser_frame">
-        <visual>
-            <geometry>
-                <cylinder radius="${chassis_width / 4}" length="${chassis_height / 4}"/>
-            </geometry>
-            <material name="green"/>
-        </visual>
-        <collision>
-            <geometry>
-                <cylinder radius="${chassis_width / 4}" length="${chassis_height / 4}"/>
-            </geometry>
-            <material name="green"/>
-        </collision>
-        <xacro:cylinder_inertia m="1.0" r="${chassis_width / 4}" h="${chassis_height / 4}" xyz="0 0 0" rpy="${pi / 2.0} 0 0" />
-    </link>
-</robot>
+/mac_remote/ws/src/macnav_description/urdf/macnav_lidar.xacro

File: remote_setup/ws/src/macnav_description/urdf/macnav_lidar.xacro (robot description, xacro)
@@ -4,5 +4,5 @@
         <parent link="chassis"/>
         <child link="laser_frame"/>
-        <origin xyz="0 0 ${9 / 8 * chassis_height }" rpy="0 0 0"/>
+        <origin xyz="0 0 ${9 / 8 * chassis_height }" rpy="0 0 ${pi / 2.0}"/>
     </joint>
     <link name="laser_frame">
